File: Schematics/RegisterFile/RegOutBuf.kicad_sch (KiCad schematic)
At the start: 0 parts

Commit message: BIG UPDATE: Schematics, PCB & updated writeup for register
Parts:
- added C36, C37, C38, C39, C40, C41, C42, C43: 0.1uF, Capacitor_SMD:C_1206_3216Metric, symbol Device:C
- added U32, U33, U34, U35, U36, U37, U38, U39: 74AHC541, Package_SO:TSSOP-20_4.4x6.5mm_P0.65mm, symbol 74xx:74AHC541
Connections:
- net ~{BUF_EN}: now also U32.1 (G1), U32.19 (G2), U33.1 (G1), U33.19 (G2), U34.1 (G1), U34.19 (G2), U35.1 (G1), U35.19 (G2), U36.1 (G1), U36.19 (G2), U37.1 (G1), U37.19 (G2), U38.1 (G1), U38.19 (G2), U39.1 (G1), U39.19 (G2)
- new net D_0: U32.2 (A0)
- new net D_1: U32.3 (A1)
- new net D_10: U33.4 (A2)
- new net D_11: U33.5 (A3)
- new net D_12: U33.6 (A4)
- new net D_13: U33.7 (A5)
- new net D_14: U33.8 (A6)
- new net D_15: U33.9 (A7)
- new net D_16: U34.2 (A0)
- new net D_17: U34.3 (A1)
- new net D_18: U34.4 (A2)
- new net D_19: U34.5 (A3)
- new net D_2: U32.4 (A2)
- new net D_20: U34.6 (A4)
- new net D_21: U34.7 (A5)
- new net D_22: U34.8 (A6)
- new net D_23: U34.9 (A7)
- new net D_24: U35.2 (A0)
- new net D_25: U35.3 (A1)
- new net D_26: U35.4 (A2)
- new net D_27: U35.5 (A3)
- new net D_28: U35.6 (A4)
- new net D_29: U35.7 (A5)
- new net D_3: U32.5 (A3)
- new net D_30: U35.8 (A6)
- new net D_31: U35.9 (A7)
- new net D_32: U36.2 (A0)
- new net D_33: U36.3 (A1)
- new net D_34: U36.4 (A2)
- new net D_35: U36.5 (A3)
- new net D_36: U36.6 (A4)
- new net D_37: U36.7 (A5)
- new net D_38: U36.8 (A6)
- new net D_39: U36.9 (A7)
- new net D_4: U32.6 (A4)
- new net D_40: U37.2 (A0)
- new net D_41: U37.3 (A1)
- new net D_42: U37.4 (A2)
- new net D_43: U37.5 (A3)
- new net D_44: U37.6 (A4)
- new net D_45: U37.7 (A5)
- new net D_46: U37.8 (A6)
- new net D_47: U37.9 (A7)
- new net D_48: U38.2 (A0)
- new net D_49: U38.3 (A1)
- new net D_5: U32.7 (A5)
- new net D_50: U38.4 (A2)
- new net D_51: U38.5 (A3)
- new net D_52: U38.6 (A4)
- new net D_53: U38.7 (A5)
- new net D_54: U38.8 (A6)
- new net D_55: U38.9 (A7)
- new net D_56: U39.2 (A0)
- new net D_57: U39.3 (A1)
- new net D_58: U39.4 (A2)
- new net D_59: U39.5 (A3)
- new net D_6: U32.8 (A6)
- new net D_60: U39.6 (A4)
- new net D_61: U39.7 (A5)
- new net D_62: U39.8 (A6)
- new net D_63: U39.9 (A7)
- new net D_7: U32.9 (A7)
- new net D_8: U33.2 (A0)
- new net D_9: U33.3 (A1)
- new net D_BUF_0: U32.18 (Y0)
- new net D_BUF_1: U32.17 (Y1)
- new net D_BUF_10: U33.16 (Y2)
- new net D_BUF_11: U33.15 (Y3)
- new net D_BUF_12: U33.14 (Y4)
- new net D_BUF_13: U33.13 (Y5)
- new net D_BUF_14: U33.12 (Y6)
- new net D_BUF_15: U33.11 (Y7)
- new net D_BUF_16: U34.18 (Y0)
- new net D_BUF_17: U34.17 (Y1)
- new net D_BUF_18: U34.16 (Y2)
- new net D_BUF_19: U34.15 (Y3)
- new net D_BUF_2: U32.16 (Y2)
- new net D_BUF_20: U34.14 (Y4)
- new net D_BUF_21: U34.13 (Y5)
- new net D_BUF_22: U34.12 (Y6)
- new net D_BUF_23: U34.11 (Y7)
- new net D_BUF_24: U35.18 (Y0)
- new net D_BUF_25: U35.17 (Y1)
- new net D_BUF_26: U35.16 (Y2)
- new net D_BUF_27: U35.15 (Y3)
- new net D_BUF_28: U35.14 (Y4)
- new net D_BUF_29: U35.13 (Y5)
- new net D_BUF_3: U32.15 (Y3)
- new net D_BUF_30: U35.12 (Y6)
- new net D_BUF_31: U35.11 (Y7)
- new net D_BUF_32: U36.18 (Y0)
- new net D_BUF_33: U36.17 (Y1)
- new net D_BUF_34: U36.16 (Y2)
- new net D_BUF_35: U36.15 (Y3)
- new net D_BUF_36: U36.14 (Y4)
- new net D_BUF_37: U36.13 (Y5)
- new net D_BUF_38: U36.12 (Y6)
- new net D_BUF_39: U36.11 (Y7)
- new net D_BUF_4: U32.14 (Y4)
- new net D_BUF_40: U37.18 (Y0)
- new net D_BUF_41: U37.17 (Y1)
- new net D_BUF_42: U37.16 (Y2)
- new net D_BUF_43: U37.15 (Y3)
- new net D_BUF_44: U37.14 (Y4)
- new net D_BUF_45: U37.13 (Y5)
- new net D_BUF_46: U37.12 (Y6)
- new net D_BUF_47: U37.11 (Y7)
- new net D_BUF_48: U38.18 (Y0)
- new net D_BUF_49: U38.17 (Y1)
- new net D_BUF_5: U32.13 (Y5)
- new net D_BUF_50: U38.16 (Y2)
- new net D_BUF_51: U38.15 (Y3)
- new net D_BUF_52: U38.14 (Y4)
- new net D_BUF_53: U38.13 (Y5)
- new net D_BUF_54: U38.12 (Y6)
- new net D_BUF_55: U38.11 (Y7)
- new net D_BUF_56: U39.18 (Y0)
- new net D_BUF_57: U39.17 (Y1)
- new net D_BUF_58: U39.16 (Y2)
- new net D_BUF_59: U39.15 (Y3)
- new net D_BUF_6: U32.12 (Y6)
- new net D_BUF_60: U39.14 (Y4)
- new net D_BUF_61: U39.13 (Y5)
- new net D_BUF_62: U39.12 (Y6)
- new net D_BUF_63: U39.11 (Y7)
- new net D_BUF_7: U32.11 (Y7)
- new net D_BUF_8: U33.18 (Y0)
- new net D_BUF_9: U33.17 (Y1)
- new net GND: C36.2, C37.2, C38.2, C39.2, C40.2, C41.2, C42.2, C43.2, U32.10 (GND), U33.10 (GND), U34.10 (GND), U35.10 (GND), U36.10 (GND), U37.10 (GND), U38.10 (GND), U39.10 (GND)
- new net VCC: C36.1, C37.1, C38.1, C39.1, C40.1, C41.1, C42.1, C43.1, U32.20 (VCC), U33.20 (VCC), U34.20 (VCC), U35.20 (VCC), U36.20 (VCC), U37.20 (VCC), U38.20 (VCC), U39.20 (VCC)
Other:
- note added: "74'541 Octal Buffers"
- note added: "Decoupling Capacitors"
