File: Schematics/CardTester/CardTester.kicad_sch (KiCad schematic)
At the start: 0 parts

Commit message: Card Tester PCB made + Register file updates
Parts:
- added C96: 10u, Capacitor_SMD:C_0805_2012Metric_Pad1.18x1.45mm_HandSolder, symbol Device:C
- added C97: 100u, Capacitor_SMD:C_0805_2012Metric_Pad1.18x1.45mm_HandSolder, symbol Device:C
- added D1: Schottky, Diode_SMD:D_0805_2012Metric_Pad1.15x1.40mm_HandSolder, symbol Device:D_Schottky
- added H1, H2, H3, H4: MountingHole, MountingHole:MountingHole_3.2mm_M3, symbol Mechanical:MountingHole
- added J1: USB_B, Connector_USB:USB_B_Lumberg_2411_02_Horizontal, symbol Connector:USB_B
- added U1: Pi_Pico, Module:RaspberryPi_Pico_Common_THT, symbol RPi Pico:Pico
- added U2: Adafruit 4711, Misc:Adafruit TLV62569 breakout (4711), symbol Misc:Adafruit TLV62569
Connections:
- new net: D1.1 (K), U1.39 (VSYS)
- new net: J1.1 (VBUS), U2.3 (Vin), U2.4 (EN)
- new net ADR_0: U1.27 (GPIO21)
- new net ADR_1: U1.26 (GPIO20)
- new net ADR_2: U1.25 (GPIO19)
- new net ADR_3: U1.24 (GPIO18)
- new net Address Decoder/~{LOAD}: U1.22 (GPIO17)
- new net Address Decoder/~{READ}: U1.21 (GPIO16)
- new net CLK: U1.32 (GPIO27_ADC1)
- new net D-BUS_0: U1.1 (GPIO0)
- new net D-BUS_1: U1.2 (GPIO1)
- new net D-BUS_10: U1.14 (GPIO10)
- new net D-BUS_11: U1.15 (GPIO11)
- new net D-BUS_12: U1.16 (GPIO12)
- new net D-BUS_13: U1.17 (GPIO13)
- new net D-BUS_14: U1.19 (GPIO14)
- new net D-BUS_15: U1.20 (GPIO15)
- new net D-BUS_2: U1.4 (GPIO2)
- new net D-BUS_3: U1.5 (GPIO3)
- new net D-BUS_4: U1.6 (GPIO4)
- new net D-BUS_5: U1.7 (GPIO5)
- new net D-BUS_6: U1.9 (GPIO6)
- new net D-BUS_7: U1.10 (GPIO7)
- new net D-BUS_8: U1.11 (GPIO8)
- new net D-BUS_9: U1.12 (GPIO9)
- new net GND: C96.2, C97.2, J1.4 (GND), J1.5 (Shield), U1.13 (GND), U1.18 (GND), U1.23 (GND), U1.28 (GND), U1.3 (GND), U1.33 (AGND), U1.38 (GND), U1.8 (GND), U2.1 (GND)
- new net LOAD: U1.29 (GPIO22)
- new net VCC: C96.1, C97.1, D1.2 (A), U2.2 (Vout)
- new net ~{CLK}: U1.31 (GPIO26_ADC0)
- no-connect marks 0 -> 19
Other:
- added sheet Address Decoder (ADR-Decode.kicad_sch)
- added sheet Control Register (CtrlReg.kicad_sch)
- added sheet DBus Buffers 1 (InBufs.kicad_sch)
- added sheet DBus Buffers 2 (InBufs.kicad_sch)
- added sheet DBus Buffers 3 (InBufs.kicad_sch)
- added sheet DBus Output Stage 1 (DOutStage.kicad_sch)
- added sheet DBus Output Stage 2 (DOutStage.kicad_sch)
- added sheet DBus Output Stage 3 (DOutStage.kicad_sch)
- added sheet DBus Registers 1 (D-FF.kicad_sch)
- added sheet DBus Registers 2 (D-FF.kicad_sch)
- added sheet DBus Registers 3 (D-FF.kicad_sch)
- added sheet IO Output Stage (IO-Out.kicad_sch)
- added sheet PCIe Connector 1 (PcieCon1.kicad_sch)
- added sheet PCIe Connector 2 (PcieCon2.kicad_sch)
- added sheet Std IO Buffers (StdIOBuf.kicad_sch)
- added sheet Std IO Registers (StdIORegs.kicad_sch)
- company: (none) -> aTan
- title: (none) -> THORN-2 Card Tester
